File: Hardware/board.brd (EAGLE design)
At the start: 170.2 x 111.3 mm, 103 parts, among them IC1 BD5229G-TR, IC4 XC6220A331MR-G, J1 FH34SRJ-24S-0.5SH_99_, J3 QWIIC_RIGHT_ANGLE, J4 112A-TAAR-R03_ATTEND, Q1 20V/4.2A/52mΩ/1.4W, Q2 20V/4.2A/52mΩ/1.4W, Q3 SI1308EDL-T1-GE3, U1 W25Q512JVEIQ, U2 ESP32-C6-WROOM-1-N8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

Commit message: Fix issues
Parts:
- moved C10_SUPERCAP 0.16 mm to (93.9, 38.0), turned to 90 degrees
- moved D1 0.13 mm to (153.1, 36.3), turned to 180 degrees
Connections:
- net DN: now also D1.4; no longer D1.1
- net DP: now also D1.6; no longer D1.3
- net GND: now also BOOT_BUTTON.1, C10_SUPERCAP.1, CHANGE_BUTTON.1, D1.2, RESET_BUTTON.1; no longer C10_SUPERCAP.2, D1.5
- net IO/BOOT: now also BOOT_BUTTON.3
- net IO/CHANGE: now also CHANGE_BUTTON.3
- net RESET: now also RESET_BUTTON.3
- net USB_D+: now also D1.1; no longer D1.4
- net USB_D-: now also D1.3; no longer D1.6
- net VBUS: now also D1.5, Q1.1; no longer D1.2
- net VRTC: now also C10_SUPERCAP.2; no longer C10_SUPERCAP.1
Routing:
- net VBUS: track 75.5 -> 94.9 mm, vias 0 -> 2
- net GND: track 664.7 -> 660.9 mm
- net RESET: track 122.3 -> 125.8 mm
- net IO/CHANGE: track 83.2 -> 86.7 mm
- net IO/BOOT: track 62.1 -> 63.8 mm
