File: Hardware/schematic.sch (EAGLE design)
At the start: 103 parts, among them IC1 BD5229G-TR, IC4 XC6220A331MR-G, J1 FH34SRJ-24S-0.5SH_99_, J2 SAMACSYS_PARTS_USB4110-GF-A, J3 QWIIC_RIGHT_ANGLE, J4 112A-TAAR-R03_ATTEND, Q1 20V/4.2A/52mΩ/1.4W, Q2 20V/4.2A/52mΩ/1.4W, Q3 SI1308EDL-T1-GE3, U1 W25Q512JVEIQ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

Commit message: Finish first stage w/o additional assigments due to deadline delay
Parts:
- C4_USB: device DeskAssistant v19 v1:EAGLE-LTSPICE_CC0402 -> DeskAssistant v19 v1:ESP32_WROVER_EAGLE-LTSPICE_CC0402
- C5_USB: value 4.7uF -> 100nF; device DeskAssistant v19 v1:EAGLE-LTSPICE_CC0402 -> DeskAssistant v19 v1:ESP32_WROVER_EAGLE-LTSPICE_CC0402
- L1: VALUE_M 68uH -> (none); VALUE_V (none) -> 68uH
- R_CAPACITOR: value (none) -> 15
- R_CL1: value (none) -> 10K
Connections:
- removed net EDP_BUSY: U2.IO3
- removed net N$2: J2.A9
- removed net N$3: J2.B4
- removed net N$30: U2.IO9
- removed net N$5: R2.2
- net 3V3: now also U1.!HOLD!/!RESET!(IO3)
- net EPD_BUSY: now also U2.IO3
- net IO/BOOT: now also U2.IO9
- net RESE': now also R2.2
- net VUSB: now also J2.A9, J2.B4
Other:
- moved on the sheet: EPD_C10, EPD_C11

Commit message: Fix issues
Connections:
- net DN: now also D1.I/O2_2; no longer D1.I/O1_1
- net DP: now also D1.I/O1_2; no longer D1.I/O2_1
- net GND: now also BOOT_BUTTON.1, C10_SUPERCAP.1, CHANGE_BUTTON.1, D1.GND, RESET_BUTTON.1; no longer C10_SUPERCAP.2, D1.VBUS
- net IO/BOOT: now also BOOT_BUTTON.3
- net IO/CHANGE: now also CHANGE_BUTTON.3
- net RESET: now also RESET_BUTTON.3
- net USB_D+: now also D1.I/O1_1; no longer D1.I/O2_2
- net USB_D-: now also D1.I/O2_1; no longer D1.I/O1_2
- net VBUS: now also D1.VBUS, Q1.G; no longer D1.GND
- net VRTC: now also C10_SUPERCAP.2; no longer C10_SUPERCAP.1
Other:
- moved on the sheet: C10_SUPERCAP, D1
Changed lines of the file:
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@@
 <part name="GND4" library="DeskAssistant v19 v1" library_urn="urn:adsk.eagle:library:47587466" deviceset="GND" device=""/>
 <part name="GND5" library="DeskAssistant v19 v1" library_urn="urn:adsk.eagle:library:47587466" deviceset="GND" device=""/>
-<part uuid="2882400009" name="D1" library="DeskAssistant v19 v1" library_urn="urn:adsk.eagle:library:47587466" deviceset="USBLC6-2SC6Y" device="" package3d_urn="urn:adsk.eagle:package:47587541/1"/>
 <part name="GND6" library="DeskAssistant v19 v1" library_urn="urn:adsk.eagle:library:47587466" deviceset="GND" device=""/>
 <part name="GND7" library="DeskAssistant v19 v1" library_urn="urn:adsk.eagle:library:47587466" deviceset="GND" device=""/>
@@
 <part name="C4_USB" library="DeskAssistant v19 v1" library_urn="urn:adsk.wipprod:fs.file:vf.rfPcC3d2T3mKPkGz0BLbYg" deviceset="ESP32_WROVER_EAGLE-LTSPICE_C" device="C0402" value="100nF"/>
 <part name="C5_USB" library="DeskAssistant v19 v1" library_urn="urn:adsk.wipprod:fs.file:vf.rfPcC3d2T3mKPkGz0BLbYg" deviceset="ESP32_WROVER_EAGLE-LTSPICE_C" device="C0402" value="100nF"/>
+<part name="D1" library="DeskAssistant v19 v1" library_urn="urn:adsk.wipprod:fs.file:vf.rfPcC3d2T3mKPkGz0BLbYg" deviceset="USBLC6-2SC6Y" device=""/>
 </parts>
 <sheets>
@@
 <attribute name="VALUE" x="124.46" y="167.64" size="1.778" layer="96" rot="R90"/>
 </instance>
-<instance part="D1" gate="G$1" x="109.22" y="187.96" smashed="yes">
-<attribute name="NAME" x="115.57" y="195.58" size="1.778" layer="95" align="center-left"/>
-<attribute name="VALUE" x="115.57" y="193.04" size="1.778" layer="96" align="center-left"/>
-</instance>
 <instance part="GND6" gate="1" x="149.86" y="185.42" smashed="yes" rot="R90">
 <attribute name="VALUE" x="152.4" y="182.88" size="1.27" layer="96" rot="R90"/>
@@
 <attribute name="VALUE" x="118.364" y="-32.639" size="1.778" layer="96"/>
 </instance>
-<instance part="C10_SUPERCAP" gate="G$1" x="127" y="-30.48" smashed="yes" rot="R90">
-<attribute name="NAME" x="135.89" y="-35.56" size="1.778" layer="95" rot="R90"/>
-<attribute name="VALUE" x="132.08" y="-30.48" size="1.778" layer="96" rot="R90"/>
+<instance part="C10_SUPERCAP" gate="G$1" x="127" y="-27.94" smashed="yes" rot="R270">
+<attribute name="NAME" x="130.81" y="-20.32" size="1.778" layer="95" rot="R270"/>
+<attribute name="VALUE" x="134.62" y="-27.94" size="1.778" layer="96" rot="R270"/>
 </instance>
 <instance part="GND42" gate="1" x="66.04" y="-33.02" smashed="yes">
@@
 <attribute name="NAME" x="151.384" y="160.401" size="1.778" layer="95"/>
 <attribute name="VALUE" x="151.384" y="155.321" size="1.778" layer="96"/>
+</instance>
+<instance part="D1" gate="G$1" x="142.24" y="182.88" smashed="yes" rot="R180">
+<attribute name="NAME" x="115.57" y="195.58" size="1.778" layer="95" rot="R180" align="center-left"/>
+<attribute name="VALUE" x="130.81" y="193.04" size="1.778" layer="96" rot="R180" align="center-left"/>
 </instance>
 </instances>
@@
 </segment>
 <segment>
-<pinref part="D1" gate="G$1" pin="GND"/>
 <wire x1="109.22" y1="185.42" x2="106.68" y2="185.42" width="0.1524" layer="91"/>
 <label x="106.68" y="185.42" size="1.27" layer="95" rot="MR0" xref="yes"/>
+<pinref part="D1" gate="G$1" pin="VBUS"/>
 </segment>
 <segment>
@@
 </segment>
 <segment>
-<wire x1="177.8" y1="175.26" x2="170.18" y2="175.26" width="0.1524" layer="91"/>
-<wire x1="170.18" y1="175.26" x2="170.18" y2="165.1" width="0.1524" layer="91"/>
-<wire x1="170.18" y1="175.26" x2="170.18" y2="185.42" width="0.1524" layer="91"/>
-<junction x="170.18" y="175.26"/>
-<label x="170.18" y="185.42" size="1.27" layer="95" rot="R90" xref="yes"/>
+<wire x1="170.18" y1="165.1" x2="170.18" y2="185.42" width="0.1524" layer="91"/>
+<label x="170.18" y="187.96" size="1.27" layer="95" rot="R90" xref="yes"/>
 <pinref part="R1_PWRUSB" gate="G$1" pin="2"/>
+<pinref part="Q1" gate="G$1" pin="G"/>
+<wire x1="187.96" y1="185.42" x2="177.8" y2="185.42" width="0.1524" layer="91"/>
+<wire x1="170.18" y1="185.42" x2="177.8" y2="185.42" width="0.1524" layer="91"/>
+<wire x1="177.8" y1="185.42" x2="177.8" y2="175.26" width="0.1524" layer="91"/>
+<junction x="170.18" y="185.42"/>
 <pinref part="D2" gate="G$0" pin="ANODE"/>
+<wire x1="170.18" y1="185.42" x2="170.18" y2="187.96" width="0.1524" layer="91"/>
+<junction x="177.8" y="185.42"/>
 </segment>
 <segment>
@@
 </segment>
 <segment>
-<pinref part="D1" gate="G$1" pin="VBUS"/>
 <wire x1="142.24" y1="185.42" x2="147.32" y2="185.42" width="0.1524" layer="91"/>
 <pinref part="GND6" gate="1" pin="GND"/>
+<pinref part="D1" gate="G$1" pin="GND"/>
 </segment>
 <segment>
@@
 <pinref part="RESET_BUTTON" gate="G$1" pin="2"/>
 <pinref part="C5" gate="G$1" pin="2"/>
+<pinref part="RESET_BUTTON" gate="G$1" pin="1"/>
+<wire x1="281.94" y1="27.94" x2="284.48" y2="27.94" width="0.1524" layer="91"/>
+<junction x="284.48" y="27.94"/>
 </segment>
 <segment>
@@
 <pinref part="BOOT_BUTTON" gate="G$1" pin="2"/>
 <pinref part="C6" gate="G$1" pin="2"/>
+<pinref part="BOOT_BUTTON" gate="G$1" pin="1"/>
+<wire x1="302.26" y1="27.94" x2="304.8" y2="27.94" width="0.1524" layer="91"/>
+<junction x="304.8" y="27.94"/>
 </segment>
 <segment>
@@
 <pinref part="CHANGE_BUTTON" gate="G$1" pin="2"/>
 <pinref part="C10" gate="G$1" pin="2"/>
+<pinref part="CHANGE_BUTTON" gate="G$1" pin="1"/>
+<wire x1="322.58" y1="27.94" x2="325.12" y2="27.94" width="0.1524" layer="91"/>
+<junction x="325.12" y="27.94"/>
 </segment>
 <segment>
@@
 <wire x1="116.84" y1="-33.02" x2="116.84" y2="-35.56" width="0.1524" layer="91"/>
 <wire x1="116.84" y1="-35.56" x2="127" y2="-35.56" width="0.1524" layer="91"/>
-<wire x1="127" y1="-35.56" x2="127" y2="-33.02" width="0.1524" layer="91"/>
-<pinref part="C10_SUPERCAP" gate="G$1" pin="2"/>
 <wire x1="127" y1="-35.56" x2="127" y2="-40.64" width="0.1524" layer="91"/>
-<junction x="127" y="-35.56"/>
 <pinref part="GND43" gate="1" pin="GND"/>
 <pinref part="C8" gate="G$1" pin="2"/>
+<pinref part="C10_SUPERCAP" gate="G$1" pin="1"/>
+<wire x1="127" y1="-33.02" x2="127" y2="-35.56" width="0.1524" layer="91"/>
+<junction x="127" y="-35.56"/>
 </segment>
 <segment>
@@
 </segment>
 <segment>
-<pinref part="D1" gate="G$1" pin="I/O2_1"/>
 <wire x1="109.22" y1="182.88" x2="106.68" y2="182.88" width="0.1524" layer="91"/>
 <label x="106.68" y="182.88" size="1.27" layer="95" rot="MR0" xref="yes"/>
+<pinref part="D1" gate="G$1" pin="I/O1_2"/>
 </segment>
 </net>
@@
 </segment>
 <segment>
-<pinref part="D1" gate="G$1" pin="I/O1_1"/>
 <wire x1="109.22" y1="187.96" x2="106.68" y2="187.96" width="0.1524" layer="91"/>
 <label x="106.68" y="187.96" size="1.27" layer="95" rot="MR0" xref="yes"/>
+<pinref part="D1" gate="G$1" pin="I/O2_2"/>
 </segment>
 </net>
@@
 <net name="USB_D-" class="0">
 <segment>
-<pinref part="D1" gate="G$1" pin="I/O1_2"/>
 <wire x1="142.24" y1="187.96" x2="142.24" y2="190.5" width="0.1524" layer="91"/>
 <wire x1="142.24" y1="190.5" x2="144.78" y2="190.5" width="0.1524" layer="91"/>
 <label x="144.78" y="190.5" size="1.27" layer="95" xref="yes"/>
+<pinref part="D1" gate="G$1" pin="I/O2_1"/>
 </segment>
 <segment>
@@
 <net name="USB_D+" class="0">
 <segment>
-<pinref part="D1" gate="G$1" pin="I/O2_2"/>
 <wire x1="142.24" y1="182.88" x2="142.24" y2="180.34" width="0.1524" layer="91"/>
 <wire x1="142.24" y1="180.34" x2="144.78" y2="180.34" width="0.1524" layer="91"/>
 <label x="144.78" y="180.34" size="1.27" layer="95" xref="yes"/>
+<pinref part="D1" gate="G$1" pin="I/O1_1"/>
 </segment>
 <segment>
@@
 <pinref part="R_CHANGE" gate="G$1" pin="1"/>
 <pinref part="C10" gate="G$1" pin="1"/>
+<pinref part="CHANGE_BUTTON" gate="G$1" pin="3"/>
+<wire x1="322.58" y1="38.1" x2="325.12" y2="38.1" width="0.1524" layer="91"/>
 </segment>
 </net>
@@
 <pinref part="R_RESET" gate="G$1" pin="1"/>
 <pinref part="C5" gate="G$1" pin="1"/>
+<pinref part="RESET_BUTTON" gate="G$1" pin="3"/>
+<wire x1="281.94" y1="38.1" x2="284.48" y2="38.1" width="0.1524" layer="91"/>
 </segment>
 </net>
@@
 <pinref part="R_BOOT" gate="G$1" pin="1"/>
 <pinref part="C6" gate="G$1" pin="1"/>
+<pinref part="BOOT_BUTTON" gate="G$1" pin="3"/>
+<wire x1="302.26" y1="38.1" x2="304.8" y2="38.1" width="0.1524" layer="91"/>
 </segment>
 <segment>
@@
 <wire x1="121.92" y1="-10.16" x2="127" y2="-10.16" width="0.1524" layer="91"/>
 <wire x1="127" y1="-10.16" x2="127" y2="-20.32" width="0.1524" layer="91"/>
-<pinref part="C10_SUPERCAP" gate="G$1" pin="1"/>
-<wire x1="127" y1="-20.32" x2="127" y2="-25.4" width="0.1524" layer="91"/>
-<junction x="127" y="-20.32"/>
 <wire x1="127" y1="-20.32" x2="116.84" y2="-20.32" width="0.1524" layer="91"/>
 <wire x1="116.84" y1="-20.32" x2="116.84" y2="-25.4" width="0.1524" layer="91"/>
@@
 <pinref part="R_CAPACITOR" gate="G$1" pin="2"/>
 <pinref part="C8" gate="G$1" pin="1"/>
-</segment>
-</net>
+<wire x1="127" y1="-20.32" x2="127" y2="-25.4" width="0.1524" layer="91"/>
+<junction x="127" y="-20.32"/>
+<pinref part="C10_SUPERCAP" gate="G$1" pin="2"/>
+</segment>
+</net>
